File: engineering/hardware/atmega328p/untitled.sch (EAGLE design)
At the start: 34 parts, among them IC1 ATMEGA328-20P, J1 5A, Q1 IRF540, Q2 IRF540, Q3 IRF540, Q4 IRF540, Q5 IRF540, Q6 IRF540, X1 16MHz

Commit message: layout ready to print
Parts:
- removed MOTOR_1, MOTOR_2, MOTOR_3, MOTOR_4, MOTOR_5, MOTOR_6: 200mA, pinhead:PINHD-1X2
- added BUTTONS: NA, pinhead:PINHD-1X5
- added C2: 1000uF, rcl:CPOL-EUE5-8.5
- added MAIN_SWITCH: 5A, pinhead:PINHD-1X2
- added MOT1, MOT2, MOT3, MOT4, MOT5, MOT6: 200mA, con-wago-500:W237-102
- added RPU_1, RPU_2, RPU_3: 10k, rcl:R-EU_0207/10
- CX1, CX2: device rcl:C-EU050-025X075 -> resistor:C-EU025-024X044
Connections:
- new net M1: IC1.(PCI19/INT1/OC2B)PD3, RG_1.1
- new net M2: IC1.(PCI21/T1/OC0B)PD5, RG_2.1
- new net M3: IC1.(PCI22/AIN0OC0A)PD6, RG_3.1
- new net M4: IC1.(PCI1/OC1A/OC1S)PB1, RG_4.1
- new net M5: IC1.(PCI2/SS/OC1B)PB2, RG_5.1
- new net M6: IC1.(PCI3/MOSI/OC2A)PB3, RG_6.1
- new net N$18: BUTTONS.2, IC1.(PCI20/XCK/T0)PD4, RPU_1.1
- new net N$19: BUTTONS.3, IC1.(PCI23/AIN1)PD7, RPU_2.1
- new net N$20: BUTTONS.4, IC1.(PCI0/ICP/CLKO)PB0, RPU_3.1
- new net N$21: J1.3, MAIN_SWITCH.1
- net +12V: now also MAIN_SWITCH.2, MOT1-2.KL, MOT2-2.KL, MOT3-2.KL, MOT4-2.KL, MOT5-2.KL, MOT6-2.KL; no longer J1.3, MOTOR_1.1, MOTOR_2.1, MOTOR_3.1, MOTOR_4.1, MOTOR_5.1, MOTOR_6.1
- net GND: now also BUTTONS.5, C2.-
- net N$11: now also MOT4-1.KL; no longer MOTOR_4.2
- net N$13: now also MOT5-1.KL; no longer MOTOR_5.2
- net N$15: now also MOT6-1.KL; no longer MOTOR_6.2
- net N$6: now also MOT1-1.KL; no longer MOTOR_1.2
- net N$7: now also MOT2-1.KL; no longer MOTOR_2.2
- net N$9: now also MOT3-1.KL; no longer MOTOR_3.2
- net VCC: now also BUTTONS.1, C2.+, RPU_1.2, RPU_2.2, RPU_3.2
Other:
- moved on the sheet: J1
